Commit message: fix(model): set X5 eef_link mass to 0.150 kg
eef_link mass was 0.0, which caused gravity compensation to
under-estimate the payload at the end-effector and produce a small
persistent drift. 0.150 kg reflects the measured gripper-side mass
on the physical arm.

Co-Authored-By: Claude Opus 4.7 <noreply@anthropic.com>

File: models/X5.urdf (robot description, URDF)
Before this commit: robot X5, 8 links, 7 joints
Links:
- link eef_link: mass 0.0 -> 0.150
